File: Hardware/Qwiic Power Switch.brd (EAGLE design)
At the start: 25.4 x 25.4 mm, 61 parts, among them J1 Qwiic Right Angle, J2 PTH, J3 Qwiic Right Angle, J4 PTH, Q1 20V/4.2A/52mΩ/1.4W, U1 74HC1G04, U2 PCA9536

Commit message: Finishing touches...
Parts:
- IN_LED: value INT -> IN_LED
- OUT_LED: value INT -> OUT_LED
Routing:
- net GND: track 49.4 -> 54.4 mm
Changed lines of the file:
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@@
 <element name="U2" library="New_Parts" package="MSOP8" value="PCA9536" x="12.7" y="12.319" smashed="yes" rot="R180">
 <attribute name="NAME" x="13.843" y="11.557" size="0.508" layer="25" rot="R180"/>
+<attribute name="PROD_ID" value="IC-15034" x="12.7" y="12.319" size="1.778" layer="27" rot="R180" display="off"/>
 </element>
 <element name="C1" library="SparkFun-Capacitors" package="0603" value="0.1uF" x="7.62" y="10.795" smashed="yes" rot="R270">
@@
 </element>
 <element name="U$10" library="Labels" package="I_SUPER2_C-()-03" value="" x="1.143" y="5.588" smashed="yes" rot="MR270"/>
-<element name="IN_LED" library="SparkFun-Jumpers" package="SMT-JUMPER_2_NC_TRACE_SILK" package3d_urn="urn:adsk.eagle:package:39281/1" value="INT" x="5.08" y="17.78" smashed="yes" rot="MR180">
+<element name="IN_LED" library="SparkFun-Jumpers" package="SMT-JUMPER_2_NC_TRACE_SILK" package3d_urn="urn:adsk.eagle:package:39281/1" value="IN_LED" x="5.08" y="17.78" smashed="yes" rot="MR180">
 <attribute name="NAME" x="4.953" y="19.812" size="0.6096" layer="26" font="vector" ratio="20" rot="MR180" align="bottom-center"/>
 </element>
@@
 <attribute name="NAME" x="6.604" y="2.159" size="0.6096" layer="25" font="vector" ratio="20" rot="R180"/>
 </element>
-<element name="OUT_LED" library="SparkFun-Jumpers" package="SMT-JUMPER_2_NC_TRACE_SILK" package3d_urn="urn:adsk.eagle:package:39281/1" value="INT" x="20.32" y="7.62" smashed="yes" rot="MR0">
+<element name="OUT_LED" library="SparkFun-Jumpers" package="SMT-JUMPER_2_NC_TRACE_SILK" package3d_urn="urn:adsk.eagle:package:39281/1" value="OUT_LED" x="20.32" y="7.62" smashed="yes" rot="MR0">
 <attribute name="NAME" x="20.701" y="5.588" size="0.6096" layer="26" font="vector" ratio="20" rot="MR0" align="bottom-center"/>
 </element>
@@
 <contactref element="U1" pad="5"/>
 <wire x1="8.89" y1="14.29" x2="8.89" y2="14.671" width="0.6096" layer="1"/>
-<wire x1="8.89" y1="14.671" x2="8.89" y2="21.59" width="0.6096" layer="1"/>
-<wire x1="8.89" y1="21.59" x2="9.525" y2="22.225" width="0.6096" layer="1"/>
-<wire x1="9.525" y1="22.225" x2="12.065" y2="22.225" width="0.6096" layer="1"/>
+<wire x1="8.89" y1="14.671" x2="8.89" y2="21.082" width="0.6096" layer="1"/>
+<wire x1="8.89" y1="21.082" x2="10.033" y2="22.225" width="0.6096" layer="1"/>
+<wire x1="10.033" y1="22.225" x2="12.065" y2="22.225" width="0.6096" layer="1"/>
 <wire x1="12.065" y1="22.225" x2="12.7" y2="22.86" width="0.6096" layer="1"/>
 <wire x1="12.7" y1="22.86" x2="12.7" y2="24.13" width="0.6096" layer="1"/>
@@
 <via x="1.27" y="11.43" extent="1-16" drill="0.3048"/>
 <via x="18.288" y="13.462" extent="1-16" drill="0.3048"/>
+<wire x1="15.24" y1="1.27" x2="15.24" y2="3.175" width="0.6096" layer="16"/>
+<wire x1="16.51" y1="4.445" x2="17.78" y2="4.445" width="0.6096" layer="16"/>
+<wire x1="15.24" y1="3.175" x2="16.51" y2="4.445" width="0.6096" layer="16"/>
 </signal>
 <signal name="N$1">
@@
 <via x="15.494" y="14.351" extent="1-16" drill="0.3048"/>
 <wire x1="15.494" y1="14.351" x2="15.113" y2="13.97" width="0.3048" layer="1"/>
-<wire x1="15.113" y1="13.97" x2="13.97" y2="13.97" width="0.3048" layer="1"/>
-<wire x1="13.081" y1="13.081" x2="12.573" y2="13.081" width="0.3048" layer="1"/>
+<wire x1="15.113" y1="13.97" x2="13.462" y2="13.97" width="0.3048" layer="1"/>
 <wire x1="11.486" y1="11.994" x2="10.45" y2="11.994" width="0.3048" layer="1"/>
-<wire x1="13.97" y1="13.97" x2="13.081" y2="13.081" width="0.3048" layer="1"/>
-<wire x1="12.573" y1="13.081" x2="11.486" y2="11.994" width="0.3048" layer="1"/>
+<wire x1="13.462" y1="13.97" x2="11.486" y2="11.994" width="0.3048" layer="1"/>
 </signal>
 <signal name="SCL">

Commit message: Version X02
Parts:
- removed U$21: (no value), OUT:OUT0
- added I2C_OUT: JUMPER-SMT_3_2-NC_TRACE_SILK, SparkFun-Jumpers:SMT-JUMPER_3_2-NC_TRACE_SILK
- added R6, R7: 2.2k, SparkFun-Resistors:0603
- added R8: 200k, SparkFun-Resistors:0603
- added U$1: (no value), IN__3:IN0
- added U$18: (no value), Labels:I_SUPER2_C-()-03
- added U3: (no value), SparkFun-IC-Comms:VSSOP_8PIN
- R2: value 1k -> 470
- U$14: device IN:IN0 -> OUT__3:OUT0
- moved J5 25.0 mm to (17.8, 1.27)
- moved J6 25.0 mm to (7.62, 24.1)
- moved U$20 24.6 mm to (7.62, 23.9), turned to 270 degrees
- moved U$25 24.6 mm to (7.62, 23.9), turned to 270 degrees
- moved U$16 24.3 mm to (17.8, 1.65), turned to 90 degrees
- moved U$24 24.3 mm to (17.8, 1.65), turned to 90 degrees
- moved J2 23.4 mm to (15.2, 1.27), turned to 0 degrees
- moved J4 23.4 mm to (10.2, 24.1), turned to 0 degrees
- moved U$12 22.1 mm to (12.7, 23.7), turned to 270 degrees
- moved U$23 22.1 mm to (12.7, 1.65), turned to 90 degrees
- moved U$4 22.1 mm to (12.7, 1.65), turned to 90 degrees
- moved U$7 22.1 mm to (12.7, 23.7), turned to 270 degrees
- moved U$14 13.5 mm to (24.1, 18.3), flipped to the bottom, turned to 270 degrees
- moved R5 5.59 mm to (15.7, 17.4)
- moved U$10 3.81 mm to (1.14, 1.78), turned to 90 degrees
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- renumbered I2C to I2C_IN
Connections:
- new net N$10: I2C_OUT.3, R6.2
- new net N$12: R8.1, U3.P7
- new net N$8: I2C_OUT.1, R7.2
- new net SCL_OUT: J3.4, J4.4, R7.1, U3.P6
- new net SDA_OUT: J3.3, J4.3, R6.1, U3.P5
- net 3.3V: now also R8.2, U3.P2
- net GND: now also U3.P1
- net GPIO0: now also U3.P8
- net SCL: now also U3.P3; no longer J3.4, J4.4
- net SDA: now also U3.P4; no longer J3.3, J4.3
- net VOUT: now also I2C_OUT.2
Routing:
- net SDA_OUT: track 0.00 -> 29.9 mm, vias 0 -> 2
- net SDA: track 59.0 -> 32.5 mm, vias 4 -> 2
- net SCL_OUT: track 0.00 -> 26.3 mm, vias 0 -> 2
- net SCL: track 52.3 -> 31.5 mm, vias 4 -> 3
- net GND: track 54.4 -> 34.9 mm
- net N$10: track 0.00 -> 5.79 mm, vias 0 -> 1
- net N$6: track 2.84 -> 6.49 mm, vias 0 -> 2
- net N$8: track 0.00 -> 3.56 mm, vias 0 -> 1
- net GPIO1: track 16.4 -> 12.9 mm, vias 1 -> 0
- net N$12: track 0.00 -> 2.93 mm
- net GPIO2: track 13.0 -> 14.9 mm, vias 0 -> 1
- net GPIO0: track 4.95 -> 6.53 mm
- net VOUT: track 35.1 -> 36.5 mm, vias 3 -> 2
- net 3.3V: track 45.1 -> 46.2 mm
- net N$5: track 7.68 -> 8.27 mm
Other:
- board text added: "X02"
- board text removed: "X01"

Commit message: Not quite finished - need to add the PCA9306 tPlace outline
Connections:
- new net GPIO3: U2.5, U3.P8
- net GPIO0: no longer U3.P8
Routing:
- net GPIO3: track 0.00 -> 6.95 mm
- net GPIO0: track 6.53 -> 3.65 mm
- net GND: vias 33 -> 32
Changed lines of the file:
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@@
 <wire x1="7.648" y1="8.735" x2="7.62" y2="8.763" width="0.3048" layer="1"/>
 <via x="12.7" y="12.446" extent="1-16" drill="0.3048"/>
-<via x="12.954" y="10.541" extent="1-16" drill="0.3048"/>
 <via x="6.477" y="14.859" extent="1-16" drill="0.3048"/>
 </signal>
@@
 <contactref element="U2" pad="1"/>
 <contactref element="U1" pad="2"/>
-<contactref element="U3" pad="P8"/>
-<wire x1="14.95" y1="11.725" x2="14.986" y2="11.689" width="0.3048" layer="1"/>
-<wire x1="12.325" y1="8.735" x2="13.15895" y2="8.735" width="0.3048" layer="1"/>
-<wire x1="13.30575" y1="8.8818" x2="13.15895" y2="8.735" width="0.3048" layer="1"/>
-<wire x1="15.936" y1="8.89" x2="15.9278" y2="8.8818" width="0.3048" layer="1"/>
-<wire x1="15.9278" y1="8.8818" x2="14.986" y2="8.8818" width="0.3048" layer="1"/>
-<wire x1="14.986" y1="8.8818" x2="13.30575" y2="8.8818" width="0.3048" layer="1"/>
-<wire x1="14.986" y1="11.689" x2="14.986" y2="8.8818" width="0.3048" layer="1"/>
+<wire x1="15.936" y1="8.89" x2="15.24" y2="8.89" width="0.3048" layer="1"/>
+<wire x1="14.95" y1="9.18" x2="14.95" y2="11.725" width="0.3048" layer="1"/>
+<wire x1="15.24" y1="8.89" x2="14.95" y2="9.18" width="0.3048" layer="1"/>
 </signal>
 <signal name="N$5">
@@
 <wire x1="11.303" y1="9.017" x2="11.645" y2="9.359" width="0.3048" layer="1"/>
 </signal>
+<signal name="GPIO3">
+<contactref element="U2" pad="5"/>
+<contactref element="U3" pad="P8"/>
+<wire x1="10.45" y1="13.675" x2="11.344" y2="13.675" width="0.3048" layer="1"/>
+<wire x1="11.344" y1="13.675" x2="11.684" y2="13.335" width="0.3048" layer="1"/>
+<wire x1="11.684" y1="11.684" x2="12.065" y2="11.303" width="0.3048" layer="1"/>
+<wire x1="12.573" y1="11.303" x2="12.827" y2="11.049" width="0.3048" layer="1"/>
+<wire x1="12.827" y1="9.237" x2="12.325" y2="8.735" width="0.3048" layer="1"/>
+<wire x1="11.684" y1="13.335" x2="11.684" y2="11.684" width="0.3048" layer="1"/>
+<wire x1="12.065" y1="11.303" x2="12.573" y2="11.303" width="0.3048" layer="1"/>
+<wire x1="12.827" y1="11.049" x2="12.827" y2="9.237" width="0.3048" layer="1"/>
+</signal>
 </signals>
