File: Hardware/Qwiic Power Switch.sch (EAGLE design)
At the start: 31 parts, among them J1 Qwiic Right Angle, J2 PTH, J3 Qwiic Right Angle, J4 PTH, Q1 20V/4.2A/52mΩ/1.4W, U1 74HC1G04, U2 PCA9536

Commit message: Finishing touches...
Parts:
- IN_LED: value INT -> IN_LED
- OUT_LED: value INT -> OUT_LED
Changed lines of the file:
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@@
 <part name="D2" library="SparkFun-LED" deviceset="LED-GREEN" device="0603" value="GREEN"/>
 <part name="R2" library="SparkFun-Resistors" deviceset="1KOHM" device="-0603-1/10W-1%" value="1k"/>
-<part name="IN_LED" library="SparkFun-Jumpers" deviceset="JUMPER-SMT_2_NC_TRACE" device="_SILK" package3d_urn="urn:adsk.eagle:package:39281/1" value="INT"/>
+<part name="IN_LED" library="SparkFun-Jumpers" deviceset="JUMPER-SMT_2_NC_TRACE" device="_SILK" package3d_urn="urn:adsk.eagle:package:39281/1" value="IN_LED"/>
 <part name="J4" library="SparkFun-Connectors" deviceset="I2C_STANDARD" device="_NO_SILK" value="PTH"/>
 <part name="GND10" library="SparkFun-PowerSymbols" deviceset="GND" device=""/>
-<part name="OUT_LED" library="SparkFun-Jumpers" deviceset="JUMPER-SMT_2_NC_TRACE" device="_SILK" package3d_urn="urn:adsk.eagle:package:39281/1" value="INT"/>
+<part name="OUT_LED" library="SparkFun-Jumpers" deviceset="JUMPER-SMT_2_NC_TRACE" device="_SILK" package3d_urn="urn:adsk.eagle:package:39281/1" value="OUT_LED"/>
 <part name="GND2" library="SparkFun-PowerSymbols" deviceset="GND" device=""/>
 <part name="SUPPLY3" library="SparkFun-PowerSymbols" deviceset="VOUT" device=""/>

Commit message: Version X02
Parts:
- removed I2C: JUMPER-SMT_3_2-NC_TRACE_SILK, SparkFun-Jumpers:JUMPER-SMT_3_2-NC_TRACE_SILK
- added I2C_IN, I2C_OUT: JUMPER-SMT_3_2-NC_TRACE_SILK, SparkFun-Jumpers:JUMPER-SMT_3_2-NC_TRACE_SILK
- added R6, R7: 2.2k, SparkFun-Resistors:2.2KOHM-0603-1/10W-1%
- added R8: 200k, SparkFun-Resistors:200KOHM-0603-1/10W-1%
- added U3: (no value), SparkFun-IC-Comms:PCA9306VSSOP_8PIN
- R2: value 1k -> 470; device SparkFun-Resistors:1KOHM-0603-1/10W-1% -> SparkFun-Resistors:470OHM-0603-1/10W-1%
Connections:
- new net N$10: I2C_OUT.3, R6.2
- new net N$12: R8.1, U3.VREF2
- new net N$8: I2C_OUT.1, R7.2
- new net SCL_OUT: J3.4, J4.4, R7.1, U3.SCL2
- new net SDA_OUT: J3.3, J4.3, R6.1, U3.SDA2
- net 3.3V: now also I2C_IN.2, R8.2, U3.VREF1; no longer I2C.2
- net GND: now also U3.GND
- net GPIO0: now also U3.EN
- net N$1: now also I2C_IN.1; no longer I2C.1
- net N$2: now also I2C_IN.3; no longer I2C.3
- net SCL: now also U3.SCL1; no longer J3.4, J4.4
- net SDA: now also U3.SDA1; no longer J3.3, J4.3
- net VOUT: now also I2C_OUT.2
Other:
- note added: "2"
- note added: "PCA9306 I C Isolation"
- note added: "PCA9536 4-Bit GPIO"
- note added: "Power Switch"
- note added: "X02"
- note removed: "X01"
- moved on the sheet: C1, C2, C3, D1, D2, IN_LED, J1, J2, J3, J4, J5, J6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

Commit message: Not quite finished - need to add the PCA9306 tPlace outline
Connections:
- new net GPIO3: U2.GPIO3, U3.EN
- net GPIO0: no longer U3.EN
Changed lines of the file:
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@@
 <segment>
 <pinref part="U3" gate="G$1" pin="VREF1"/>
-<wire x1="165.1" y1="106.68" x2="162.56" y2="106.68" width="0.1524" layer="91"/>
+<wire x1="167.64" y1="106.68" x2="162.56" y2="106.68" width="0.1524" layer="91"/>
 <pinref part="SUPPLY16" gate="G$1" pin="3.3V"/>
 <wire x1="162.56" y1="106.68" x2="162.56" y2="111.76" width="0.1524" layer="91"/>
@@
 <segment>
 <pinref part="U3" gate="G$1" pin="GND"/>
-<wire x1="165.1" y1="99.06" x2="162.56" y2="99.06" width="0.1524" layer="91"/>
+<wire x1="167.64" y1="99.06" x2="162.56" y2="99.06" width="0.1524" layer="91"/>
 <pinref part="GND12" gate="1" pin="GND"/>
 <wire x1="162.56" y1="99.06" x2="162.56" y2="96.52" width="0.1524" layer="91"/>
@@
 <segment>
 <pinref part="U3" gate="G$1" pin="SDA1"/>
-<wire x1="165.1" y1="101.6" x2="160.02" y2="101.6" width="0.1524" layer="91"/>
+<wire x1="167.64" y1="101.6" x2="160.02" y2="101.6" width="0.1524" layer="91"/>
 <label x="160.02" y="101.6" size="1.27" layer="95" rot="R180" xref="yes"/>
 </segment>
@@
 <segment>
 <pinref part="U3" gate="G$1" pin="SCL1"/>
-<wire x1="165.1" y1="104.14" x2="160.02" y2="104.14" width="0.1524" layer="91"/>
+<wire x1="167.64" y1="104.14" x2="160.02" y2="104.14" width="0.1524" layer="91"/>
 <label x="160.02" y="104.14" size="1.27" layer="95" rot="R180" xref="yes"/>
 </segment>
@@
 <wire x1="137.16" y1="55.88" x2="134.62" y2="55.88" width="0.1524" layer="91"/>
 </segment>
-<segment>
-<pinref part="U3" gate="G$1" pin="EN"/>
-<wire x1="195.58" y1="109.22" x2="195.58" y2="116.84" width="0.1524" layer="91"/>
-<wire x1="195.58" y1="116.84" x2="187.96" y2="116.84" width="0.1524" layer="91"/>
-<label x="187.96" y="116.84" size="1.27" layer="95" rot="R180" xref="yes"/>
-</segment>
 </net>
 <net name="N$5" class="0">
@@
 <segment>
 <pinref part="U3" gate="G$1" pin="SDA2"/>
-<wire x1="195.58" y1="101.6" x2="200.66" y2="101.6" width="0.1524" layer="91"/>
+<wire x1="193.04" y1="101.6" x2="200.66" y2="101.6" width="0.1524" layer="91"/>
 <label x="200.66" y="101.6" size="1.27" layer="95" xref="yes"/>
 </segment>
@@
 <segment>
 <pinref part="U3" gate="G$1" pin="SCL2"/>
-<wire x1="195.58" y1="104.14" x2="200.66" y2="104.14" width="0.1524" layer="91"/>
+<wire x1="193.04" y1="104.14" x2="200.66" y2="104.14" width="0.1524" layer="91"/>
 <label x="200.66" y="104.14" size="1.27" layer="95" xref="yes"/>
 </segment>
@@
 <segment>
 <pinref part="U3" gate="G$1" pin="VREF2"/>
-<wire x1="195.58" y1="106.68" x2="200.66" y2="106.68" width="0.1524" layer="91"/>
+<wire x1="193.04" y1="106.68" x2="200.66" y2="106.68" width="0.1524" layer="91"/>
 <pinref part="R8" gate="G$1" pin="1"/>
 <wire x1="200.66" y1="106.68" x2="200.66" y2="111.76" width="0.1524" layer="91"/>
 </segment>
 </net>
+<net name="GPIO3" class="0">
+<segment>
+<pinref part="U2" gate="U1" pin="GPIO3"/>
+<wire x1="193.04" y1="147.32" x2="195.58" y2="147.32" width="0.1524" layer="91"/>
+<label x="195.58" y="147.32" size="1.27" layer="95" xref="yes"/>
+</segment>
+<segment>
+<pinref part="U3" gate="G$1" pin="EN"/>
+<wire x1="193.04" y1="109.22" x2="193.04" y2="116.84" width="0.1524" layer="91"/>
+<wire x1="193.04" y1="116.84" x2="187.96" y2="116.84" width="0.1524" layer="91"/>
+<label x="187.96" y="116.84" size="1.27" layer="95" rot="R180" xref="yes"/>
+</segment>
+</net>
